File: PCB/Auth75.kicad_sch (KiCad schematic)
At the start: 209 parts, among them CN1 S2B-PH-SM4-TB, Q1 MMBT3904-C20526, Q2 MMBT3904-C20526, Q3 MMBT3904-C20526, Q4 SS8550_C8542, Q5 FS8205A_C2830320, SW1 EC11E15244G1, U1 RASPBERRY PI PICO 2W, U2 SL2.1S, U3 DW01A_C351410, U4 MCP73831T-2ACI/OT, U5 PCA9536DGKR

Commit message: uhhh
Parts:
- S1, S10, S11, S12, S13, S14, S15, S16, S17, S18, S19, S2, S20, S21, S22, S23, S24, S25, S26, S27, S3, S30, S31, S32, S33, S34, S35, S36, S37, S38, S39, S4, S40, S41, S44, S45, S46, S47, S48, S49, S5, S50, S51, S52, S53, S54, S57, S58, S59, S6, S60, S61, S62, S63, S64, S65, S66, S68, S7, S73, S74, S75, S76, S77, S78, S8, S9: footprint Switch_Keyboard_Hotswap_Kailh:SW_Hotswap_Kailh_MX_1.00u -> Switch_Keyboard_Hotswap_Kailh:SW_Hotswap_Kailh_MX
- S28: footprint Switch_Keyboard_Hotswap_Kailh:SW_Hotswap_Kailh_MX_2.00u -> Switch_Keyboard_Hotswap_Kailh:SW_Hotswap_Kailh_MX
- S29, S42: footprint Switch_Keyboard_Hotswap_Kailh:SW_Hotswap_Kailh_MX_1.50u -> Switch_Keyboard_Hotswap_Kailh:SW_Hotswap_Kailh_MX
- S43, S67: footprint Switch_Keyboard_Hotswap_Kailh:SW_Hotswap_Kailh_MX_1.75u -> Switch_Keyboard_Hotswap_Kailh:SW_Hotswap_Kailh_MX
- S55, S56: footprint Switch_Keyboard_Hotswap_Kailh:SW_Hotswap_Kailh_MX_2.25u -> Switch_Keyboard_Hotswap_Kailh:SW_Hotswap_Kailh_MX
- S69, S70, S71: footprint Switch_Keyboard_Hotswap_Kailh:SW_Hotswap_Kailh_MX_1.25u -> Switch_Keyboard_Hotswap_Kailh:SW_Hotswap_Kailh_MX
- S72: footprint Switch_Keyboard_Hotswap_Kailh:SW_Hotswap_Kailh_MX_6.25u -> Switch_Keyboard_Hotswap_Kailh:SW_Hotswap_Kailh_MX
